File: FULL BOARD/FULL BOARD/_autosave-FULL BOARD.kicad_sch (KiCad schematic)
At the start: 72 parts, among them J1 PJ-036AH-SMT-TR, J2 Micro_SD_Card, J3 Conn_01x04_Male, SW1 SW_Push, U1 LD1117S33TR_SOT223, U2 STM32H743VITx, Y1 16Mhz

Commit message: schematic done
Parts:
- removed FB1: FerriteBead, symbol Device:FerriteBead
- removed J3: Conn_01x04_Male, symbol Connector:Conn_01x04_Male
- removed Y1: 16Mhz, symbol Device:Crystal_GND24
- added FL1: BLM15GA750SZ1D, footprints:BEADC1005X55N, symbol BLM15GA750SZ1D:BLM15GA750SZ1D
- added J4: 5019514000, footprints:CON_5019514000, symbol 2024-09-26_21-43-55:5019514000
- added J5: 61201021621, footprints:CONN_61201021621_WRE, symbol 2024-09-27_18-41-52:61201021621
- added R4, R5, R6, R7: 1k, Resistor_SMD:R_0805_2012Metric, symbol Device:R_US
- added Y1: ABLS7M2-16.000MHZ-D-2Y-T, footprints:XTAL_ABLS7M2-16.000MHZ-D-2Y-T, symbol ABLS7M2-16.000MHZ-D-2Y-T:ABLS7M2-16.000MHZ-D-2Y-T
- C1, C15, C4: footprint (none) -> Capacitor_SMD:C_0805_2012Metric
- C10, C11, C12, C13, C14, C16, C17, C18, C19, C20, C5, C6, C9: footprint (none) -> Capacitor_SMD:C_0402_1005Metric
- C2, C7, C8: footprint Capacitor_SMD:C_0805_2012Metric_Pad1.15x1.40mm_HandSolder -> Capacitor_SMD:C_0402_1005Metric
- C3: footprint (none) -> Capacitor_SMD:C_0603_1608Metric
- D1, D10, D11, D12, D13, D14, D15, D16, D17, D18, D19, D2, D20, D3, D4, D5, D6, D7, D8, D9: footprint ScottoKeebs_Components:Diode_DO-35 -> Keyboard footprint:Diode_DO-35
- R1, R2, R3: footprint Resistor_SMD:R_0805_2012Metric_Pad1.15x1.40mm_HandSolder -> Resistor_SMD:R_0805_2012Metric
- S1, S10, S11, S12, S13, S14, S15, S16, S17, S18, S19, S2, S20, S3, S4, S5, S6, S7, S8, S9: footprint ScottoKeebs_MX:MX_PCB_1.00u -> Keyboard footprint:MX_PCB_1.00u
Connections:
- net +3.3V: now also FL1.2
- net +3.3VA: now also FL1.1
- net Col 1: now also R4.2; no longer S1.1, S13.1, S17.1, S5.1, S9.1
- net Col 2: now also R5.2; no longer S10.1, S14.1, S18.1, S2.1, S6.1
- net Col 3: now also R6.2; no longer S11.1, S15.1, S19.1, S3.1, S7.1
- net Col 4: now also R7.2; no longer S12.1, S16.1, S20.1, S4.1, S8.1
- net GND: now also J5.3, J5.4
- net HSE_IN: now also Y1.1
- net HSE_OUT: now also Y1.2
- net NRST: now also J5.1
- net SWC: now also J5.6
- net SWDIO: now also J5.2
- net LCD_CS: now reaches U2.28 (PA4)
- net LCD_CS: now also J4.5
- net LCD_SCK: now reaches U2.29 (PA5)
- net LCD_SCK: now also J4.8
- net LCD_MISO: now reaches U2.30 (PA6)
- net LCD_MISO: now also J4.6
- net LCD_MOSI: now reaches U2.31 (PA7)
- net LCD_MOSI: now also J4.7
- new net: R5.1, S10.1, S14.1, S18.1, S2.1, S6.1
- new net: R6.1, S11.1, S15.1, S19.1, S3.1, S7.1
- new net: R4.1, S1.1, S13.1, S17.1, S5.1, S9.1
- new net: R7.1, S12.1, S16.1, S20.1, S4.1, S8.1
Other:
- moved on the sheet: C1, C10, C11, C12, C14, C15, C16, C17, C18, C19, C20, C3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
