File: FULL BOARD/FULL BOARD/FULL BOARD.kicad_sch (KiCad schematic)
At the start: 113 parts, among them IC1 TAS5760LDAP, J1 PJ-036AH-SMT-TR, J2 Micro_SD_Card, J3 B2B-PH-K-S, J4 5019514000, J5 61201021621, J6 B2B-PH-K-S, SW1 PTS645SK50SMTR92LFS, U1 LD1117S33TR_SOT223, U2 STM32H743VITx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

Commit message: parts moved
Connections:
- net Wait: now reaches U2.32 (PC4)
- net Wait: now also J4.9
- no-connect marks 96 -> 94
Changed lines of the file:
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@@
 	)
 	(no_connect
-		(at 138.43 158.75)
-	)
-	(no_connect
 		(at 128.27 196.85)
 	)
@@
 	)
 	(no_connect
+		(at 138.43 130.81)
+	)
+	(no_connect
 		(at 138.43 173.99)
 	)
@@
 	)
 	(no_connect
-		(at 304.8 190.5)
-	)
-	(no_connect
 		(at 238.76 190.5)
 	)
@@
 	)
 	(no_connect
-		(at 138.43 130.81)
-	)
-	(no_connect
 		(at 138.43 250.19)
 	)
@@
 	(wire
 		(pts
+			(xy 129.54 158.75) (xy 138.43 158.75)
+		)
+		(stroke
+			(width 0)
+			(type default)
+		)
+	)
+	(wire
+		(pts
 			(xy 246.38 326.39) (xy 256.54 326.39)
 		)
@@
 	(wire
 		(pts
+			(xy 304.8 176.53) (xy 304.8 190.5)
+		)
+		(stroke
+			(width 0)
+			(type default)
+		)
+	)
+	(wire
+		(pts
 			(xy 128.27 201.93) (xy 138.43 201.93)
 		)
@@
 		)
 	)
+	(global_label "Wait"
+		(shape input)
+		(at 129.54 158.75 180)
+		(fields_autoplaced yes)
+		(effects
+			(font
+				(size 1.27 1.27)
+			)
+			(justify right)
+		)
+		(property "Intersheetrefs" "${INTERSHEET_REFS}"
+			(at 122.6239 158.75 0)
+			(effects
+				(font
+					(size 1.27 1.27)
+				)
+				(justify right)
+				(hide yes)
+			)
+		)
+	)
 	(global_label "I2S_CK"
 		(shape input)
@@
 				(hide yes)
 			)
+		)
+	)
+	(global_label "Wait"
+		(shape input)
+		(at 304.8 176.53 90)
+		(fields_autoplaced yes)
+		(effects
+			(font
+				(size 1.27 1.27)
+			)
+			(justify left)
+		)
+		(property "Intersheetrefs" "${INTERSHEET_REFS}"
+			(at 304.8 169.6139 90)
+			(effects
+				(font
+					(size 1.27 1.27)
+				)
+				(justify left)
+				(hide yes)
+			)

Commit message: changed reset footprint
Parts:
- SW1: footprint push button custom:SW4_PTS645SK50SMTR92LFS_CNK -> Reset Switch:SW_PTS645SK50SMTR92LFS
Changed lines of the file:
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@@
 			)
 		)
-		(property "Footprint" "push button custom:SW4_PTS645SK50SMTR92LFS_CNK"
+		(property "Footprint" "Reset Switch:SW_PTS645SK50SMTR92LFS"
 			(at 34.29 142.24 0)
 			(effects

Commit message: change SD
Parts:
- removed J2: Micro_SD_Card, Connector_Card:microSD_HC_Molex_47219-2001, symbol Connector:Micro_SD_Card
- added J2: MEM2080-00-128-00-A, MEM20800012800A, symbol Second SD Card:MEM2080-00-128-00-A
Connections:
- net +3.3V: now also J2.4 (VDD)
- net GND: now also J2.6 (VSS)
- net SD_CLK: now also J2.5 (CLK)
- net SD_CS: now also J2.2 (CD/DAT3)
- net SD_DI: now also J2.3 (CMD)
- net SD_DO: now also J2.7 (DAT0)
- no-connect marks 94 -> 99
Changed lines of the file:
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@@
 	)
 	(no_connect
-		(at 30.48 304.8)
+		(at 322.58 152.4)
 	)
 	(no_connect
-		(at 283.21 154.94)
+		(at 30.48 304.8)
 	)
 	(no_connect
@@
 	)
 	(no_connect
+		(at 322.58 144.78)
+	)
+	(no_connect
 		(at 128.27 199.39)
 	)
@@
 	)
 	(no_connect
-		(at 283.21 137.16)
+		(at 281.94 137.16)
+	)
+	(no_connect
+		(at 322.58 139.7)
 	)
 	(no_connect
@@
 	)
 	(no_connect
+		(at 322.58 137.16)
+	)
+	(no_connect
 		(at 269.24 190.5)
 	)
@@
 	)
 	(no_connect
+		(at 322.58 149.86)
+	)
+	(no_connect
 		(at 138.43 135.89)
 	)
@@
 	)
 	(no_connect
+		(at 322.58 147.32)
+	)
+	(no_connect
 		(at 181.61 163.83)
 	)
@@
 	)
 	(no_connect
+		(at 322.58 142.24)
+	)
+	(no_connect
 		(at 292.1 190.5)
 	)
@@
 	)
 	(no_connect
-		(at 326.39 160.02)
-	)
-	(no_connect
 		(at 138.43 168.91)
 	)
@@
 	(wire
 		(pts
-			(xy 274.32 139.7) (xy 283.21 139.7)
+			(xy 274.32 139.7) (xy 281.94 139.7)
 		)
 		(stroke
@@
 	(wire
 		(pts
-			(xy 274.32 147.32) (xy 283.21 147.32)
+			(xy 274.32 147.32) (xy 281.94 147.32)
 		)
 		(stroke
@@
 	(wire
 		(pts
-			(xy 264.16 149.86) (xy 283.21 149.86)
+			(xy 264.16 149.86) (xy 281.94 149.86)
 		)
 		(stroke
@@
 	(wire
 		(pts
-			(xy 274.32 152.4) (xy 283.21 152.4)
+			(xy 274.32 152.4) (xy 281.94 152.4)
 		)
 		(stroke
@@
 	(wire
 		(pts
-			(xy 254 144.78) (xy 283.21 144.78)
+			(xy 254 144.78) (xy 281.94 144.78)
 		)
 		(stroke
@@
 	(wire
 		(pts
-			(xy 274.32 142.24) (xy 283.21 142.24)
+			(xy 274.32 142.24) (xy 281.94 142.24)
 		)
 		(stroke
@@
 	)
 	(symbol
+		(lib_id "Second SD Card:MEM2080-00-128-00-A")
+		(at 281.94 137.16 0)
+		(unit 1)
+		(exclude_from_sim no)
+		(in_bom yes)
+		(on_board yes)
+		(dnp no)
+		(fields_autoplaced yes)
+		(property "Reference" "J2"
+			(at 302.26 129.54 0)
+			(effects
+				(font
+					(size 1.27 1.27)
+				)
+			)
+		)
+		(property "Value" "MEM2080-00-128-00-A"
+			(at 302.26 132.08 0)
+			(effects
+				(font
+					(size 1.27 1.27)
+				)
+			)
+		)
+		(property "Footprint" "MEM20800012800A"
+			(at 318.77 232.08 0)
+			(effects
+				(font
+					(size 1.27 1.27)
+				)
+				(justify left top)
+				(hide yes)
+			)
+		)
+		(property "Datasheet" "https://gct.co/files/drawings/mem2080.pdf?v=a9dd5643-7d1c-4e6b-bf46-1b82bcb8595f"
+			(at 318.77 332.08 0)
+			(effects
+				(font
+					(size 1.27 1.27)
+				)
+				(justify left top)
+				(hide yes)
+			)
+		)
+		(property "Description" "Memory Card Connectors Micro SD, Push Push, SMT, Card Entry Normal, 1.28 mm profile"
+			(at 281.94 137.16 0)
+			(effects
+				(font
+					(size 1.27 1.27)
+				)
+				(hide yes)
+			)
+		)
+		(property "Height" "1.48"
+			(at 318.77 532.08 0)
+			(effects
+				(font
+					(size 1.27 1.27)
+				)
+				(justify left top)
+				(hide yes)
+			)
+		)
+		(property "Mouser Part Number" "640-MEM2080-0012800A"
+			(at 318.77 632.08 0)
+			(effects
+				(font
+					(size 1.27 1.27)
+				)
+				(justify left top)
+				(hide yes)
+			)
+		)
+		(property "Mouser Price/Stock" "https://www.mouser.co.uk/ProductDetail/GCT/MEM2080-00-128-00-A?qs=vvQtp7zwQdPJXzpf1SnYug%3D%3D"
+			(at 318.77 732.08 0)
+			(effects
+				(font
+					(size 1.27 1.27)
+				)
+				(justify left top)
+				(hide yes)
+			)
+		)
+		(property "Manufacturer_Name" "GCT (GLOBAL CONNECTOR TECHNOLOGY)"
+			(at 318.77 832.08 0)
+			(effects
+				(font
+					(size 1.27 1.27)
+				)
+				(justify left top)
+				(hide yes)
+			)
+		)
+		(property "Manufacturer_Part_Number" "MEM2080-00-128-00-A"
+			(at 318.77 932.08 0)
+			(effects
+				(font
+					(size 1.27 1.27)
+				)
+				(justify left top)
+				(hide yes)
+			)
+		)
+		(pin "4"
+		)
+		(pin "6"
+		)
+		(pin "7"
+		)
+		(pin "MP1"
+		)
+		(pin "MP3"
+		)
+		(pin "MP2"
+		)
+		(pin "DSW1"
+		)
+		(pin "8"
+		)
+		(pin "1"
+		)
+		(pin "3"
+		)
+		(pin "DSW2"
+		)
+		(pin "MP4"
+		)
+		(pin "2"
+		)
+		(pin "5"
+		)
+		(instances
+			(project ""
+				(path "/df550598-5349-47af-a3f3-2a2a958bedd4"
+					(reference "J2")
+					(unit 1)
+				)
+			)
+		)
+	)
+	(symbol
 		(lib_id "Device:C")
 		(at 31.75 113.03 0)
@@
 					(unit 1)
 				)
-			)
-		)
-	)
-	(symbol
-		(lib_id "Connector:Micro_SD_Card")
-		(at 306.07 144.78 0)
-		(unit 1)
-		(exclude_from_sim no)
-		(in_bom yes)
-		(on_board yes)
-		(dnp no)
-		(fields_autoplaced yes)
-		(property "Reference" "J2"
-			(at 306.705 125.73 0)
-			(effects
-				(font
-					(size 1.27 1.27)
-				)
-			)
-		)
-		(property "Value" "Micro_SD_Card"
-			(at 306.705 128.27 0)
-			(effects
-				(font
-					(size 1.27 1.27)
-				)
-			)
-		)
-		(property "Footprint" "Connector_Card:microSD_HC_Molex_47219-2001"
-			(at 335.28 137.16 0)
-			(effects
-				(font
-					(size 1.27 1.27)
-				)
-				(hide yes)
-			)
-		)
-		(property "Datasheet" "http://katalog.we-online.de/em/datasheet/693072010801.pdf"
-			(at 306.07 144.78 0)
-			(effects
-				(font
-					(size 1.27 1.27)
-				)
-				(hide yes)
-			)
-		)
-		(property "Description" "Micro SD Card Socket"
-			(at 306.07 144.78 0)
-			(effects
-				(font
-					(size 1.27 1.27)
-				)
-				(hide yes)
-			)
-		)
-		(pin "3"
-		)
-		(pin "2"
-		)
-		(pin "9"
-		)
-		(pin "8"
-		)
-		(pin "5"
-		)
-		(pin "1"
-		)
-		(pin "4"
-		)
-		(pin "6"
-		)
-		(pin "7"
-		)
-		(instances
-			(project ""
-				(path "/df550598-5349-47af-a3f3-2a2a958bedd4"
-					(reference "J2")
-					(unit 1)
-				)

Commit message: most feedback changes made
Parts:
- removed C17: 100nF, Capacitor_SMD:C_0805_2012Metric, symbol Device:C
- removed C20: 1uF, Capacitor_SMD:C_0805_2012Metric, symbol Device:C
- removed FL1, FL2: BLM15GA750SZ1D, Ferrite Bead:BEADC1005X55N, symbol BLM15GA750SZ1D:BLM15GA750SZ1D
- added D22, D26, D27, D28, D29, D30, D31, D32, D33: BZX84Cxx, Package_TO_SOT_SMD:SOT-23, symbol Diode:BZX84Cxx
- added R21, R22, R23, R24, R25, R26, R27, R28, R29: 100, Resistor_SMD:R_0805_2012Metric, symbol Device:R_US
- C18: value 10nF -> 100nF
- C3: value 10uF -> 4.7uF
- J2: footprint MEM20800012800A -> Second SD card:MEM20800012800A
Connections:
- net +3.3V: no longer U2.20 (VREF+)
- net +3.3VA: now also U2.20 (VREF+)
- net Col 1: now also D22.1 (A), R21.2; no longer R4.2
- net Col 2: now also D26.1 (A), R22.2; no longer R5.2
- net Col 3: now also D27.1 (A), R23.2; no longer R6.2
- net Col 4: now also D28.1 (A), R24.2; no longer R7.2
- net GND: now also IC1.11 (SPK_GAIN0), IC1.12 (SPK_GAIN1), D22.3 (K), D26.3 (K), D27.3 (K), D28.3 (K), D29.3 (K), D30.3 (K), D31.3 (K), D32.3 (K), D33.3 (K); no longer C18.2, C19.2
- net GNDA: now also C18.2, C19.2
- net Row 1: now also D33.1 (A), R29.2; no longer D1.1 (K), D2.1 (K), D3.1 (K), D4.1 (K)
- net Row 2: now also D32.1 (A), R28.2; no longer D5.1 (K), D6.1 (K), D7.1 (K), D8.1 (K)
- net Row 3: now also D31.1 (A), R27.2; no longer D10.1 (K), D11.1 (K), D12.1 (K), D9.1 (K)
- net Row 4: now also D30.1 (A), R26.2; no longer D13.1 (K), D14.1 (K), D15.1 (K), D16.1 (K)
- net Row 5: now also D29.1 (A), R25.2; no longer D17.1 (K), D18.1 (K), D19.1 (K), D20.1 (K)
- new net: D5.1 (K), D6.1 (K), D7.1 (K), D8.1 (K), R28.1
- new net: R21.1, R4.2
- new net: D13.1 (K), D14.1 (K), D15.1 (K), D16.1 (K), R26.1
- new net: R22.1, R5.2
- new net: R24.1, R7.2
- new net: D17.1 (K), D18.1 (K), D19.1 (K), D20.1 (K), R25.1
- new net: D10.1 (K), D11.1 (K), D12.1 (K), D9.1 (K), R27.1
- new net: D1.1 (K), D2.1 (K), D3.1 (K), D4.1 (K), R29.1
- new net: R23.1, R6.2
- no-connect marks 99 -> 92
Other:
- moved on the sheet: C21, C22, C23, C24, C25, C26, C27, C28, C29, C30, C31, C32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
